File: SoilHealthSensorIntegration/_autosave-SoilHealthSensorIntegration.kicad_sch (KiCad schematic)
At the start: 20 parts, among them J1 USB_C_Receptacle_USB2.0_14P, U1 ESP32-S2-SOLO-N4, U3 LP87334DRHDR

Commit message: fixed schem
Parts:
- added C10, C8, C9: C, symbol Device:C
- added L2: L, symbol Device:L
- added R10, R9: R, symbol Device:R
- added U4: LM5166DRCT, DRC0010J, symbol 2025-03-20_05-27-29:LM5166DRCT
- R3, R4: value 5.1K -> R
Connections:
- net +5V: no longer R3.1, R4.2
- net GND: now also R3.2, C9.2, U4.10 (GND), U4.11 (PAD), U4.5 (RT), U4.9 (HYS)
- net at J1.A5 (CC1), R7.2: no longer R4.1
- net at J1.B5 (CC2), R8.2: no longer R3.2
- new net: C10.1, R10.2
- new net: R4.1, R9.2, U4.8 (VOUT_FB)
- new net: C9.1, U4.4 (SS)
- new net: L2.1, U4.1 (SW)
- new net: C8.1, U4.2 (VIN), U4.7 (EN)
- new net: R3.1, U4.3 (ILIM)
